Commit message: built goat urdf with xacro

File: goat_description/robots/goat.urdf (robot description, URDF)
Before this commit: robot goat, 15 links, 14 joints
Links:
- added link velodyne, mass 0.01; visual mesh filename=package://velodyne_description/meshes/VLP16_scan.dae
- added link velodyne_base_link, mass 0.83; collision cylinder length=0.0717 radius=0.0516; visual mesh filename=package://velodyne_description/meshes/VLP16_base_1.dae
Joints:
- added joint velodyne_base_mount_joint: type fixed, parent top_box, child velodyne_base_link, origin xyz=0 0 0.084 rpy=0 0 0
- added joint velodyne_base_scan_joint: type fixed, parent velodyne_base_link, child velodyne, origin xyz=0 0 0.0377 rpy=0 0 0
